File: hw/sch_pcb/RTC02.kicad_pcb (KiCad board)
At the start: 2 copper layers, 40.1 x 40.1 mm, 21 parts, among them J1 JUMP_5X2, J2 JUMP2_2x1, J3 JUMP_2x1, J4 JUMP_2x1, J5 JUMP_2x1, J6 JUMP_2x1, M1 HOLE, M2 HOLE, M3 HOLE, M4 HOLE, SW1 SW_PUSH, U1 PCF85263A, Y1 ABS07-120-32.768KHZ-T

Commit message: Update project to KiCAD7.
Other:
- net class Default removed
